File: PCB/Anson's Keyboard PCB.kicad_pcb (KiCad board)
At the start: 2 copper layers, 352.5 x 136.4 mm, 373 parts, among them SW1 ESC, SW10 F9, SW11 F10, SW12 F11, SW13 F12, SW14 PRNT, SW15 TILDE, SW16 1, SW17 2, SW18 3, SW19 4, SW2 F1, SW20 5, SW21 6, SW22 7, SW23 8, SW24 9, SW25 0, SW26 HYPHEN, SW27 EQUAL, SW28 BACKSPACE, SW29 TAB, SW3 F2, SW30 Q, SW31 W, SW32 E, SW33 R, SW34 T, SW35 Y, SW36 U, SW37 I, SW38 O, SW39 P, SW4 F3, SW40 LEFTBRACK, SW41 RIGHTBRACK, SW42 BACKSLASH, SW43 CAPS, SW44 A, SW45 S, SW46 D, SW47 F, SW48 G, SW49 H, SW5 F4, SW50 J, SW51 K, SW52 L, SW53 SEMICOL, SW54 QUOTE, SW55 ENTER, SW56 DELETE, SW57 LSHIFT, SW58 Z, SW59 X, SW6 F5, SW60 C, SW61 V, SW62 B, SW63 N, SW64 M, SW65 COMMA, SW66 PERIOD, SW67 SLASH, SW68 RSHIFT, SW69 UP, SW7 F6, SW70 END, SW71 LCTRL, SW72 LWIN, SW73 LALT, SW74 SPACE, SW75 RALT, SW76 RWIN, SW77 MENU, SW78 RCTRL, SW79 LEFT, SW8 F7, SW80 DOWN, SW81 RIGHT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

Commit message: Updated PCB to use hotswap
Rewired everything to use hotswap sockets instead of direct switch soldering
Parts:
- SW1, SW10, SW11, SW12, SW13, SW14, SW15, SW16, SW17, SW18, SW19, SW2, SW20, SW21, SW22, SW23, SW24, SW25, SW26, SW27, SW3, SW30, SW31, SW32, SW33, SW34, SW35, SW36, SW37, SW38, SW39, SW4, SW40, SW41, SW44, SW45, SW46, SW47, SW48, SW49, SW5, SW50, SW51, SW52, SW53, SW54, SW56, SW58, SW59, SW6, SW60, SW61, SW62, SW63, SW64, SW65, SW66, SW67, SW69, SW7, SW70, SW79, SW8, SW80, SW81, SW82, SW83, SW84, SW85, SW86, SW87, SW9: footprint Library:SW_Cherry_MX_1.00u_PCB -> hotSwap:SW_Hotswap_Kailh_MX_Plated_1.00u
- SW28: footprint Library:SW_Cherry_MX_2.00u_PCB -> hotSwap:SW_Hotswap_Kailh_MX_Plated_2.00u
- SW29, SW42: footprint Library:SW_Cherry_MX_1.50u_PCB -> hotSwap:SW_Hotswap_Kailh_MX_Plated_1.50u
- SW43: footprint Library:SW_Cherry_MX_1.75u_PCB -> hotSwap:SW_Hotswap_Kailh_MX_Plated_1.75u
- SW55, SW57: footprint Library:SW_Cherry_MX_2.25u_PCB -> hotSwap:SW_Hotswap_Kailh_MX_Plated_2.25u
- SW68: footprint Library:SW_Cherry_MX_2.75u_PCB -> hotSwap:SW_Hotswap_Kailh_MX_Plated_2.75u
- SW71, SW72, SW73, SW75, SW76, SW77, SW78: footprint Library:SW_Cherry_MX_1.25u_PCB -> hotSwap:SW_Hotswap_Kailh_MX_Plated_1.25u
- SW74: footprint Library:SW_Cherry_MX_6.25u_PCB -> hotSwap:SW_Hotswap_Kailh_MX_Plated_6.25u
- U3: footprint RF_Module:ESP32-S3-WROOM-1 -> Library:ESP32-S3-WROOM-1
- moved D1 12.3 mm to (48.3, 107.7), turned to 180 degrees
- moved D71 4.43 mm to (38.0, 201.7)
- moved D78 4.16 mm to (299.5, 203.9)
- moved D77 4.16 mm to (275.7, 204.1)
- moved D72 3.98 mm to (62.2, 201.9)
- moved D2 3.63 mm to (79.7, 96.4)
- moved D4 3.17 mm to (112.7, 97.9)
- moved D15 3.00 mm to (39.4, 124.8)
- moved D16 3.00 mm to (58.4, 124.8)
- moved D17 3.00 mm to (77.5, 124.8)
- moved D18 3.00 mm to (96.5, 124.8)
- moved D19 3.00 mm to (115.6, 124.8)
- moved D20 3.00 mm to (134.6, 124.8)
- moved D21 3.00 mm to (153.7, 124.8)
- moved D22 3.00 mm to (172.7, 124.8)
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Routing:
- net +5V: track 154.9 -> 387.3 mm, vias 44 -> 130
- net ROW 3: track 338.7 -> 376.4 mm, vias 15 -> 17
- net ROW 1: track 344.5 -> 379.7 mm
- net GND: track 667.0 -> 688.0 mm, vias 149 -> 158
- net COL 2: track 152.3 -> 166.8 mm
- net Net-(LED36-DOUT): track 26.9 -> 14.5 mm
- net COL 9: track 359.5 -> 371.4 mm, vias 4 -> 6
- net COL 4: track 186.1 -> 177.9 mm
- net Net-(D1-A): track 3.63 -> 11.7 mm
- net ROW 4: track 393.2 -> 400.4 mm
- net Net-(D75-A): track 3.63 -> 10.5 mm, vias 0 -> 2
- net COL 6: track 246.7 -> 240.8 mm, vias 6 -> 4
- net Net-(LED10-DIN): track 30.8 -> 25.4 mm
- net COL 3: track 158.5 -> 163.7 mm, vias 2 -> 3
- net COL 7: track 298.3 -> 303.2 mm, vias 5 -> 6
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