File: PCB/Anson's Keyboard PCB.kicad_pcb (KiCad board)
At the start: 2 copper layers, 352.5 x 136.4 mm, 373 parts, among them SW1 ESC, SW10 F9, SW11 F10, SW12 F11, SW13 F12, SW14 PRNT, SW15 TILDE, SW16 1, SW17 2, SW18 3, SW19 4, SW2 F1, SW20 5, SW21 6, SW22 7, SW23 8, SW24 9, SW25 0, SW26 HYPHEN, SW27 EQUAL, SW28 BACKSPACE, SW29 TAB, SW3 F2, SW30 Q, SW31 W, SW32 E, SW33 R, SW34 T, SW35 Y, SW36 U, SW37 I, SW38 O, SW39 P, SW4 F3, SW40 LEFTBRACK, SW41 RIGHTBRACK, SW42 BACKSLASH, SW43 CAPS, SW44 A, SW45 S, SW46 D, SW47 F, SW48 G, SW49 H, SW5 F4, SW50 J, SW51 K, SW52 L, SW53 SEMICOL, SW54 QUOTE, SW55 ENTER, SW56 DELETE, SW57 LSHIFT, SW58 Z, SW59 X, SW6 F5, SW60 C, SW61 V, SW62 B, SW63 N, SW64 M, SW65 COMMA, SW66 PERIOD, SW67 SLASH, SW68 RSHIFT, SW69 UP, SW7 F6, SW70 END, SW71 LCTRL, SW72 LWIN, SW73 LALT, SW74 SPACE, SW75 RALT, SW76 RWIN, SW77 MENU, SW78 RCTRL, SW79 LEFT, SW8 F7, SW80 DOWN, SW81 RIGHT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

Commit message: Multiple Changes
Added more PCB mounting holes
Changed PCB mounting hole size to M2
Added updated PCB Gerber
Added updated PCB 3D model
Updated assembled .f3z [AWS outage broke Autodesk, currently can't export f3z] and .STEP for new mounting points and changes
Updated BOM for additional screws and heatset inserts
CaseStand.step now uses screws, which is more reliable than slide-and-click mount
Removed branding on printed parts
Split large parts for printability
Updated README with new assets
Routing:
- net COL 6: track 240.8 -> 241.9 mm
- net Net-(LED79-DOUT): track 47.5 -> 48.2 mm
- net COL 13: track 520.2 -> 520.1 mm, vias 6 -> 5
Other:
- outline, holes or cut-outs redrawn
